File: doc/clock.sch (EAGLE design)
At the start: 29 parts, among them IC1 MEGA8-P, T1 BC547, T2 BC547, T3 BC547, T4 BC547

Commit message: Latest corrections
Parts:
- added LED1: (no value), led:LED5MM
- added R14, R15, R16: 10k, resistor:R-EU_0207/10
- added R17: 220, resistor:R-EU_0207/10
- added SV2: (no value), con-harting-ml:ML10L
- Q1: value (none) -> 8MHz
- SV1: device con-harting-ml:ML10L -> con-harting-ml:ML26L
Connections:
- removed net N$25: IC1.PB1(OC1A), SV1.6
- removed net N$26: IC1.PC4(ADC4/SDA), SV1.4
- removed net N$27: IC1.PC5(ADC5/SCL), SV1.2
- new net RXD: IC1.PD1(TXD), SV1.10
- new net TXD: IC1.PD0(RXD), SV1.8
- net GND: now also R14.1, R15.1, R16.1, R17.1, SV1.25, SV2.9; no longer SV1.10
- net N$1: now also IC1.PB0(ICP), R5.1; no longer IC1.PD7(AIN1), R2.1
- net N$17: now also R14.2, SV1.11, SV2.5; no longer IC1.PD0(RXD), SV1.3
- net N$18: now also R15.2, SV1.13, SV2.3; no longer IC1.PD1(TXD), SV1.5
- net N$19: now also R16.2, SV1.15, SV2.1; no longer IC1.PD2(INT0), SV1.7
- net N$2: now also IC1.PB4(MISO); no longer IC1.PD6(AIN0)
- net N$20: now also LED1.A, SV1.12; no longer IC1.PD3(INT1), SV1.9
- net N$22: now also LED1.C, R17.2; no longer IC1.PB0(ICP), SV1.8
- net N$3: now also IC1.PB3(MOSI/OC2); no longer IC1.PD5(T1)
- net N$4: now also IC1.PB5(SCK), R2.1; no longer R5.1
- net N$5: now also IC1.PB1(OC1A), R9.1; no longer IC1.PC0(ADC0), R6.1
- net N$6: now also IC1.PB2(SS/OC1B), R8.1; no longer IC1.PC1(ADC1), R7.1
- net N$7: now also IC1.PC0(ADC0), R7.1; no longer IC1.PC2(ADC2), R8.1
- net N$8: now also IC1.PC1(ADC1), R6.1; no longer IC1.PC3(ADC3), R9.1
- net SEG_0: now also IC1.PC5(ADC5/SCL); no longer IC1.PB2(SS/OC1B)
- net SEG_1: now also IC1.PC4(ADC4/SDA); no longer IC1.PB3(MOSI/OC2)
- net SEG_2: now also IC1.PC3(ADC3); no longer IC1.PB4(MISO)
- net SEG_3: now also IC1.PC2(ADC2); no longer IC1.PB5(SCK)
- net VCC: now also SV2.2
Other:
- note added: "Button board"
- note added: "Clock display"
- note added: "Raspberry PI GPIO"
- moved on the sheet: C1, C2, C3, C4, C5, IC1, LD1, LD2, LD3, LD4, Q1, R1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
